File: LiDAR Scanner.kicad_sch (KiCad schematic)
At the start: 4 parts, among them P1 USB_C_Plug_USB2.0, U1 STM32F415RGTx, U2 ICM-42688-P, U3 AP2112K-3.3

Commit message: finished v1 schematic
Parts:
- removed P1: USB_C_Plug_USB2.0, symbol Connector:USB_C_Plug_USB2.0
- removed U1: STM32F415RGTx, Package_QFP:LQFP-64_10x10mm_P0.5mm, symbol MCU_ST_STM32F4:STM32F415RGTx
- added C1, C11: 10uF, symbol Device:C_Small
- added C10: 47uF, symbol Device:C_Small
- added C12, C16, C17, C2, C3, C5, C6, C7, C8, C9: 100nF, symbol Device:C_Small
- added C13, C14: 22pF, symbol Device:C_Small
- added C15: 4.7uF, symbol Device:C_Small
- added C4: 10nF, symbol Device:C_Small
- added D1, D2: ESD5Zxx, Diode_SMD:D_SOD-523, symbol Diode:ESD5Zxx
- added D3: GREEN, symbol Device:LED
- added F1: Polyfuse_Small, symbol Device:Polyfuse_Small
- added FB1: FerriteBead_Small, symbol Device:FerriteBead_Small
- added J1: USB_C_Receptacle_USB2.0_14P, symbol Connector:USB_C_Receptacle_USB2.0_14P
- added J2: PWR TEST, symbol Connector:Conn_01x04_Pin
- added J3: UART DEBUG, symbol Connector:Conn_01x03_Pin
- added J5: SWD, symbol Connector:Conn_01x04_Pin
- added J6: GENERAL DEBUG, symbol Connector_Generic:Conn_02x06_Counter_Clockwise
- added R1, R2: 5.1k, symbol Device:R_Small_US
- added R3, R4: 10k, symbol Device:R_Small_US
- added R5, R8: 0, symbol Device:R_Small_US
- added R7: 270, symbol Device:R_Small_US
- added SW1: RESET, symbol Switch:SW_Push
- added SW2: BOOT, symbol Switch:SW_Push
- added U1: (no value), symbol LiDAR Scanner:RPLiDAR_A1_I/O
- added U4: USBLC6-2SC6, Package_TO_SOT_SMD:SOT-23-6, symbol Power_Protection:USBLC6-2SC6
- added U5: STM32F411CEUx, Package_DFN_QFN:QFN-48-1EP_7x7mm_P0.5mm_EP5.6x5.6mm, symbol MCU_ST_STM32F4:STM32F411CEUx
- added Y2: 8MHz, symbol Device:Crystal_GND2_Small
Connections:
- net SPI1_MISO: now reaches U2.1 (AP_SDO/AP_AD0)
- net SPI1_MISO: now also J6.11 (Pin_11), U5.16 (PA6)
- net SPI1_CS: now reaches U2.12 (AP_CS)
- net SPI1_CS: now also J6.9 (Pin_9), U5.18 (PB0)
- net SPI1_SCK: now reaches U2.13 (AP_SCL/AP_SCLK)
- net SPI1_SCK: now also J6.10 (Pin_10), U5.15 (PA5)
- net SPI1_MOSI: now reaches U2.14 (AP_SDA/AP_SDIO/AP_SDI)
- net SPI1_MOSI: now also J6.12 (Pin_12), U5.17 (PA7)
- net INT (EXTI): now reaches U2.4 (INT1/INT)
- net INT (EXTI): now also U5.43 (PB7)
- net 3.3V: now reaches U2.5 (VDDIO)
- net 3.3V: now also U2.8 (VDD), C12.1, C16.1, C17.1, C3.2, C5.1, C6.1, C7.1, C8.1, D3.2 (A), FB1.1, J2.3 (Pin_3), J5.1 (Pin_1), J6.3 (Pin_3), R3.1, R5.2, SW2.1, U5.1 (VBAT), U5.24 (VDD), U5.36 (VDD), U5.48 (VDD)
- net GND: now reaches U2.6 (GND)
- net GND: now also U2.7 (RESV), U2.9 (INT2/FSYNC/CLKIN), U3.2 (GND), C1.1, C10.2, C11.1, C12.2, C13.2, C14.2, C15.1, C16.2, C17.2, C2.1, C3.1, C4.1, C5.2, C6.2, C7.2, C8.2, C9.2, D1.2 (A), D2.2 (A), J1.A1 (GND), J1.A12 (GND), J1.B1 (GND), J1.B12 (GND), J1.SH (SHIELD), J2.4 (Pin_4), J3.3 (Pin_3), J5.2 (Pin_2), J6.1 (Pin_1), R1.1, R2.1, R4.2, R7.1, SW1.1, U1.4 (DGND), U1.7 (MGND), U4.2 (GND), U5.23 (VSS), U5.35 (VSS), U5.47 (VSS), U5.49 (VSS), U5.8 (VSSA), Y2.2
- net VCC: now reaches U3.1 (VIN)
- net VCC: now also U3.3 (EN), C1.2, C2.2, C9.1, F1.2, J2.2 (Pin_2), J6.2 (Pin_2), R8.2, U1.1 (VCC_5), U4.5 (VBUS)
- net at U3.5 (VOUT): now also C11.2, R5.1
- new net: C15.2, U5.22 (VCAP1)
- new net: C14.1, U5.6 (PH1), Y2.3
- new net: C13.1, U5.5 (PH0), Y2.1
- new net: C10.1, R8.1, U1.5 (VMOTO)
- new net: C4.2, FB1.2, U5.9 (VDDA)
- new net: D3.1 (K), R7.2
- new net: J1.A7 (D-), J1.B7 (D-), U4.1 (I/O1)
- new net: J1.A6 (D+), J1.B6 (D+), U4.3 (I/O2)
- new net BOOT0: R4.1, SW2.2, U5.44 (BOOT0)
- new net CC1: J1.A5 (CC1), R1.2
- new net CC2: J1.B5 (CC2), R2.2
- new net D+: U4.4 (I/O2), U5.33 (PA12)
- new net D-: U4.6 (I/O1), U5.32 (PA11)
- new net DEBUG_A: J6.6 (Pin_6), U5.26 (PB13)
- new net DEBUG_B: J6.8 (Pin_8), U5.27 (PB14)
- new net DEBUG_C: J6.7 (Pin_7), U5.28 (PB15)
- new net NRST: R3.2, SW1.2, U5.7 (NRST)
- new net PWM: U1.6 (PWM), U5.29 (PA8)
- new net SWCLK: D2.1 (K), J5.4 (Pin_4), U5.37 (PA14)
- new net SWDIO: D1.1 (K), J5.3 (Pin_3), U5.34 (PA13)
- new net UART1_RX: J6.5 (Pin_5), U1.3 (RX), U5.30 (PA9)
- new net UART1_TX: J6.4 (Pin_4), U1.2 (TX), U5.31 (PA10)
- new net UART2_RX: J3.2 (Pin_2), U5.13 (PA3)
- new net UART2_TX: J3.1 (Pin_1), U5.12 (PA2)
- new net VIN: F1.1, J1.A4 (VBUS), J1.A9 (VBUS), J1.B4 (VBUS), J1.B9 (VBUS), J2.1 (Pin_1)
Other:
- note added: "Header for Debugging"
- note added: "IMU"
- note added: "MCU"
- note added: "RPLiDAR Interface"
- note added: "USB & Power"
- note added: "enable/disable motor"
- title: Handheld 2D LiDAR scanner -> (none)
- moved on the sheet: U2, U3
