File: LiDAR Scanner.kicad_sch (KiCad schematic)
At the start: 42 parts, among them J1 USB_C_Receptacle_USB2.0_14P, J2 PWR TEST, J3 UART DEBUG, J5 SWD, J6 GENERAL DEBUG, SW1 RESET, SW2 BOOT, U2 ICM-42688-P, U3 AP2112K-3.3, U4 USBLC6-2SC6, U5 STM32F411CEUx, Y2 8MHz

Commit message: Added stitching vias, electrolytic caps, final design
Parts:
- removed C12: 100nF, symbol Device:C_Small
- removed J1: USB_C_Receptacle_USB2.0_14P, symbol Connector:USB_C_Receptacle_USB2.0_14P
- removed R4: 10k, symbol Device:R_Small_US
- removed R8: 0, symbol Device:R_Small_US
- removed SW2: BOOT, symbol Switch:SW_Push
- removed Y2: 8MHz, symbol Device:Crystal_GND2_Small
- added C16: 2.2uF, Capacitor_SMD:C_0603_1608Metric_Pad1.08x0.95mm_HandSolder, symbol Device:C_Small
- added C8: 10uF, Capacitor_SMD:C_0603_1608Metric_Pad1.08x0.95mm_HandSolder, symbol Device:C_Small
- added FB2: 1A, low DCR, 600R @ 100MHz, Inductor_SMD:L_0805_2012Metric_Pad1.05x1.20mm_HandSolder, symbol Device:FerriteBead_Small
- added J1: USB4215-03-A, LiDAR:GCT_USB4215-03-A_REVA, symbol Connector:USB_C_Receptacle_USB2.0_16P
- added J4: GPIO DEBUG, Connector_PinHeader_2.54mm:PinHeader_1x05_P2.54mm_Vertical, symbol Connector:Conn_01x05_Pin
- added R6: 10k, Capacitor_SMD:C_0603_1608Metric_Pad1.08x0.95mm_HandSolder, symbol Device:R_Small_US
- added R7: 10k, Resistor_SMD:R_0603_1608Metric_Pad0.98x0.95mm_HandSolder, symbol Device:R_Small_US
- added SW2: SW_Nidec_CAS-120A1, Button_Switch_SMD:Nidec_Copal_CAS-120A, symbol Switch:SW_Nidec_CAS-120A1
- added Y1: 8MHz, LiDAR:ABM3B_ABR, symbol Device:Crystal_GND24_Small
- C1, C2, R1, R2: footprint (none) -> Capacitor_SMD:C_0603_1608Metric_Pad1.08x0.95mm_HandSolder
- C10: renamed from C3; value 100nF -> 0.1uF; footprint (none) -> Capacitor_SMD:C_0603_1608Metric_Pad1.08x0.95mm_HandSolder
- C11: renamed from C13; footprint (none) -> Capacitor_SMD:C_0603_1608Metric_Pad1.08x0.95mm_HandSolder
- C12: renamed from C14; footprint (none) -> Capacitor_SMD:C_0603_1608Metric_Pad1.08x0.95mm_HandSolder
- C13: renamed from C15; footprint (none) -> Capacitor_SMD:C_0603_1608Metric_Pad1.08x0.95mm_HandSolder
- C14: renamed from C17; value 100nF -> 10nF; footprint (none) -> Capacitor_SMD:C_0603_1608Metric_Pad1.08x0.95mm_HandSolder
- C15: renamed from C16; footprint (none) -> Capacitor_SMD:C_0603_1608Metric_Pad1.08x0.95mm_HandSolder
- C17: renamed from C9; value 100nF -> 22uF; footprint (none) -> LiDAR:PCAP_6.3x3-ELECT_NCA-L
- C18: renamed from C10; footprint (none) -> LiDAR:PCAP_6.3x3-ELECT_NCA-L
- C3: renamed from C11; footprint (none) -> Capacitor_SMD:C_0603_1608Metric_Pad1.08x0.95mm_HandSolder
- C4: renamed from C8; footprint (none) -> Capacitor_SMD:C_0603_1608Metric_Pad1.08x0.95mm_HandSolder
- C5: renamed from C6; footprint (none) -> Capacitor_SMD:C_0603_1608Metric_Pad1.08x0.95mm_HandSolder
- C6: renamed from C7; footprint (none) -> Capacitor_SMD:C_0603_1608Metric_Pad1.08x0.95mm_HandSolder
- C7: renamed from C5; footprint (none) -> Capacitor_SMD:C_0603_1608Metric_Pad1.08x0.95mm_HandSolder
- C9: renamed from C4; footprint (none) -> Capacitor_SMD:C_0603_1608Metric_Pad1.08x0.95mm_HandSolder
- D3: footprint (none) -> LED_SMD:LED_0805_2012Metric_Pad1.15x1.40mm_HandSolder
- F1: footprint (none) -> Fuse:Fuse_0805_2012Metric_Pad1.15x1.40mm_HandSolder
- FB1: footprint (none) -> Inductor_SMD:L_0603_1608Metric_Pad1.05x0.95mm_HandSolder
- J2, J5: footprint (none) -> Connector_PinHeader_2.54mm:PinHeader_1x04_P2.54mm_Vertical
- J3: footprint (none) -> Connector_PinHeader_2.54mm:PinHeader_1x03_P2.54mm_Vertical
- J6: footprint (none) -> Connector_PinHeader_2.54mm:PinHeader_2x06_P2.54mm_Vertical
- R3: renamed from R5; footprint (none) -> Capacitor_SMD:C_0603_1608Metric_Pad1.08x0.95mm_HandSolder
- R4: renamed from R7; footprint (none) -> Capacitor_SMD:C_0603_1608Metric_Pad1.08x0.95mm_HandSolder
- R5: renamed from R3; footprint (none) -> Capacitor_SMD:C_0603_1608Metric_Pad1.08x0.95mm_HandSolder
- SW1: footprint (none) -> LiDAR:SW_B3F-1000_OMR
- U1: footprint (none) -> LiDAR:CONN_22035075_MOL
- U2: footprint LGA14_2P5X3X0P91_TDK -> LiDAR:LGA14_2P5X3X0P91_TDK
Connections:
- net 3.3V: now also C16.1, C8.1, J4.1 (Pin_1), SW2.1 (C); no longer C10.2
- net BOOT0: now also R7.2
- net CC1: now also J1.A5 (CC1)
- net CC2: now also J1.B5 (CC2)
- net DEBUG_A: now also U5.39 (PB3), J4.2 (Pin_2); no longer J6.6 (Pin_6), U5.26 (PB13)
- net DEBUG_B: now also U5.40 (PB4), J4.3 (Pin_3); no longer J6.8 (Pin_8), U5.27 (PB14)
- net DEBUG_C: now also U5.41 (PB5), J4.4 (Pin_4); no longer J6.7 (Pin_7), U5.28 (PB15)
- net GND: now also C10.2, J6.6 (Pin_6), J6.7 (Pin_7), J6.8 (Pin_8), U1.3 (MGND), C16.2, C8.2, J1.A1 (GND), J1.A12 (GND), J1.B1 (GND), J1.B12 (GND), J1.SH (SHIELD), J4.5 (Pin_5), SW2.3 (A), Y1.2 (G), Y1.4 (G); no longer C10.1, U1.4 (DGND)
- net INT (EXTI): now also U5.18 (PB0); no longer U5.43 (PB7)
- net NRST: now also C10.1, R6.2; no longer R5.2, SW1.2
- net PWM: now also U1.2 (PWM), U5.21 (PB10); no longer U1.6 (PWM), U5.29 (PA8)
- net SPI1_CS: now also U5.14 (PA4); no longer U5.18 (PB0)
- net UART1_RX: now also J6.4 (Pin_4), U1.5 (RX); no longer J6.5 (Pin_5), U1.3 (RX)
- net UART1_TX: now also J6.5 (Pin_5), U1.6 (TX); no longer J6.4 (Pin_4), U1.2 (TX)
- net VCC: now also U1.4 (VCC_5), FB2.2; no longer U1.1 (VCC_5)
- net VIN: now also J1.A4 (VBUS), J1.A9 (VBUS), J1.B4 (VBUS), J1.B9 (VBUS)
- net at C12.1, U5.6 (PH1): now also Y1.1
- net at C11.1, U5.5 (PH0): now also Y1.3
- net at C18.1: now also U1.1 (VMOTO), FB2.1; no longer U1.5 (VMOTO)
- net UIN_N: now reaches U4.1 (I/O1)
- net UIN_N: now also J1.A7 (D-), J1.B7 (D-)
- net UIN_P: now reaches U4.3 (I/O2)
- net UIN_P: now also J1.A6 (D+), J1.B6 (D+)
- net D+ renamed USB_P
- net D- renamed USB_N
- new net: R5.2, R6.1, SW1.2
- new net: R7.1, SW2.2 (B)
- no-connect marks 0 -> 19
Other:
- note added: "ABM3B"
- note added: "Crystal: ABM3B-8.000MHZ-B2-T Button: B3F-1002"
- note added: "Headers for Debugging"
- note added: "UZG1C470MCL1GB"
- note added: "UZG1V220MCL1GB"
- note removed: "Header for Debugging"
- note removed: "enable/disable motor"
- moved on the sheet: C10, J6, R5, SW1
