File: LiDAR_Scanner_v1/LiDAR Scanner.kicad_pcb (KiCad board)
At the start: 4 copper layers, 82 x 82 mm, 49 parts, among them J1 USB4215-03-A, J2 PWR TEST, J3 UART DEBUG, J4 GPIO DEBUG, J5 SWD, J6 GENERAL DEBUG, SW1 RESET, SW2 SW_Nidec_CAS-120A1, U2 ICM-42688-P, U3 AP2112K-3.3, U4 USBLC6-2SC6, U5 STM32F411CEUx, Y1 8MHz

Commit message: Added more detailed photos
Routing:
- net GND: vias 311 -> 308
Changed lines of the file:
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@@
-	)
-	(via
-		(at 186.2 120.4)
-		(size 0.6)
-		(drill 0.3)
-		(layers "F.Cu" "B.Cu")
-		(free yes)
-		(net "GND")
 	)
 	(via
@@
 	)
 	(via
-		(at 176.2 120.4)
-		(size 0.6)
-		(drill 0.3)
-		(layers "F.Cu" "B.Cu")
-		(free yes)
-		(net "GND")
-	)
-	(via
 		(at 174.244 97.536)
 		(size 0.45)
@@
 		(size 0.6)
 		(drill 0.3)
-		(layers "F.Cu" "B.Cu")
-		(free yes)
-		(net "GND")
-	)
-	(via
-		(at 184.2 90.4)
-		(size 0.6)
-		(drill 0.3)
